File: PCB/brutalist_01/brutalist_01.kicad_sch (KiCad schematic)
At the start: 123 parts, among them SW1 A Sync, SW10 A ND, SW11 A Prelisten, SW12 A Jump Inc, SW13 A Jump Pos, SW14 A Play, SW15 A Intro, SW16 A Loop Inc, SW17 A Reloop, SW18 Select 2, SW19 B Sync, SW2 A Jump Dec, SW20 B Jump Dec, SW21 B Jump Neg, SW22 B Loop Dec, SW23 B Loop, SW24 B Pitch, SW25 B Nudge, SW26 B Scrub, SW27 B ND, SW28 B Prelisten, SW29 B Jump Inc, SW3 A Jump Neg, SW30 B Jump Pos, SW31 B Play, SW32 B Intro, SW33 B Loop Inc, SW34 B Reloop, SW4 A Loop Dec, SW5 A Loop, SW6 A Pitch, SW7 A Nudge, SW8 A Scrub, SW9 Select 1, U0 CD74HC4067M, U1 CD74HC4067M, U2 CD74HC4067M, U3 CD74HC4067M, U4 ProMicro, U5 Nano Every

Commit message: add footprints
Parts:
- C1, C10, C11, C12, C13, C14, C15, C16, C2, C3, C4, C5, C6, C7, C8, C9: footprint (none) -> Capacitor_THT:C_Disc_D10.0mm_W2.5mm_P5.00mm
- D1, D2, D3, D4: footprint (none) -> LED_THT:LED_D5.0mm
- R1, R10, R11, R12, R13, R14, R15, R16, R17, R18, R19, R2, R20, R21, R22, R23, R24, R25, R26, R27, R28, R29, R3, R30, R31, R32, R33, R34, R35, R36, R37, R38, R39, R4, R40, R41, R42, R43, R44, R45, R46, R47, R48, R5, R6, R7, R8, R9: footprint (none) -> Resistor_THT:R_Axial_DIN0207_L6.3mm_D2.5mm_P10.16mm_Horizontal
- RV1, RV10, RV11, RV12, RV14, RV15, RV2, RV3, RV4, RV5, RV6, RV8, RV9: footprint (none) -> Potentiometer_THT:Potentiometer_Alps_RK09K_Single_Vertical
- SW1, SW10, SW11, SW12, SW13, SW14, SW15, SW16, SW17, SW19, SW2, SW20, SW21, SW22, SW23, SW27, SW28, SW29, SW3, SW30, SW31, SW32, SW33, SW34, SW4, SW5: footprint (none) -> Button_Switch_Keyboard:SW_Cherry_MX_1.00u_PCB
- SW18, SW9: footprint (none) -> Rotary_Encoder:RotaryEncoder_Alps_EC11E-Switch_Vertical_H20mm
- SW24, SW25, SW26, SW6, SW7, SW8: footprint (none) -> Rotary_Encoder:RotaryEncoder_Alps_EC12E_Vertical_H20mm
Connections:
- net MUX0_07: now also R18.1, SW9.S1
- net MUX1_07: now also R29.1, SW18.S1
- removed net xxx: R18.1, R29.1, SW18.S1, SW9.S1
- no-connect marks 41 -> 39

Commit message: add custom mx footprint
Parts:
- RV13, RV7: footprint (none) -> Custom:ALPS RS60112
- SW1, SW10, SW11, SW12, SW13, SW14, SW15, SW16, SW17, SW19, SW2, SW20, SW21, SW22, SW23, SW27, SW28, SW29, SW3, SW30, SW31, SW32, SW33, SW34, SW4, SW5: footprint Button_Switch_Keyboard:SW_Cherry_MX_1.00u_PCB -> Custom:SW_Cherry_MX_1.00u_PCB_edit
