File: PCB/brutalist_01/brutalist_01.kicad_pcb (KiCad board)
At the start: 2 copper layers, 123 parts, among them SW1 A Sync, SW10 A ND, SW11 A Prelisten, SW12 A Jump Inc, SW13 A Jump Pos, SW14 A Play, SW15 A Intro, SW16 A Loop Inc, SW17 A Reloop, SW18 Select 2, SW19 B Sync, SW2 A Jump Dec, SW20 B Jump Dec, SW21 B Jump Neg, SW22 B Loop Dec, SW23 B Loop, SW24 B Pitch, SW25 B Nudge, SW26 B Scrub, SW27 B ND, SW28 B Prelisten, SW29 B Jump Inc, SW3 A Jump Neg, SW30 B Jump Pos, SW31 B Play, SW32 B Intro, SW33 B Loop Inc, SW34 B Reloop, SW4 A Loop Dec, SW5 A Loop, SW6 A Pitch, SW7 A Nudge, SW8 A Scrub, SW9 Select 1, U0 CD74HC4067M, U1 CD74HC4067M, U2 CD74HC4067M, U3 CD74HC4067M, U4 ProMicro, U5 Nano Every

Commit message: create traces for basic infrastructure
Routing:
- net NE_14: track 0.00 -> 382.8 mm, vias 0 -> 2
- net NE_15: track 0.00 -> 364.2 mm, vias 0 -> 2
- net NE_13: track 0.00 -> 312.2 mm, vias 0 -> 2
- net NE_12: track 0.00 -> 308.3 mm, vias 0 -> 2
- net S2: track 0.00 -> 300.0 mm, vias 0 -> 2
- net NE_01: track 0.00 -> 274.0 mm, vias 0 -> 1
- net S0: track 0.00 -> 266.1 mm, vias 0 -> 4
- net A1: track 0.00 -> 265.5 mm, vias 0 -> 2
- net S3: track 0.00 -> 262.3 mm, vias 0 -> 2
- net NE_02: track 0.00 -> 259.6 mm, vias 0 -> 1
- net S1: track 0.00 -> 256.1 mm, vias 0 -> 2
- net NE_11: track 0.00 -> 256.0 mm, vias 0 -> 2
- net NE_00: track 0.00 -> 247.4 mm, vias 0 -> 1
- net A3: track 0.00 -> 243.4 mm, vias 0 -> 4
- net A2: track 0.00 -> 222.8 mm, vias 0 -> 2
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Other:
- board outline added: 142.5 x 266 mm

Commit message: finish routing
Parts:
- added REF**: MountingHole_3.2mm_M3, MountingHole:MountingHole_3.2mm_M3, F.Cu at (213.8, 61.8)
- added REF**: MountingHole_3.2mm_M3, MountingHole:MountingHole_3.2mm_M3, F.Cu at (80.8, 61.8)
- added REF**: MountingHole_3.2mm_M3, MountingHole:MountingHole_3.2mm_M3, F.Cu at (213.8, 327.8)
- added REF**: MountingHole_3.2mm_M3, MountingHole:MountingHole_3.2mm_M3, F.Cu at (80.8, 327.8)
Routing:
- net VCC: track 0.00 -> 1536.6 mm, vias 0 -> 6
- net MUX1_07: track 0.00 -> 191.6 mm
- net MUX0_07: track 0.00 -> 151.9 mm, vias 0 -> 3
- net MUX3_05: track 0.00 -> 150.0 mm, vias 0 -> 2
- net MUX3_06: track 0.00 -> 139.6 mm, vias 0 -> 2
- net MUX2_05: track 0.00 -> 138.4 mm, vias 0 -> 6
- net MUX1_02: track 0.00 -> 125.9 mm, vias 0 -> 2
- net MUX2_13: track 0.00 -> 118.6 mm
- net MUX3_13: track 0.00 -> 108.4 mm, vias 0 -> 2
- net MUX3_04: track 0.00 -> 101.4 mm, vias 0 -> 2
- net MUX1_03: track 0.00 -> 99.1 mm, vias 0 -> 2
- net MUX0_02: track 0.00 -> 98.3 mm, vias 0 -> 2
- net MUX0_03: track 0.00 -> 95.6 mm, vias 0 -> 2
- net MUX1_11: track 0.00 -> 95.0 mm, vias 0 -> 2
- net MUX1_12: track 0.00 -> 93.2 mm, vias 0 -> 2
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- added copper zone on B.Cu, net GND
- added copper zone on F.Cu, net GND
Other:
- board size 142.5 x 266 mm -> 142.5 x 275.5 mm
- board text added: "BREMEN 2023 REV. 0"
- board text added: "GOOD ENOUGH STILL BETTER THAN YOURS"
- board text added: "JLCJLCJLCJLC"
